Commit message: [URDF] corrected link origin to joint origin

File: code/ros-drivers/scoomatic_description/urdf/scoomatic.urdf (robot description, URDF)
Before this commit: robot scoomatic, 7 links, 6 joints
Joints:
- joint base_to_imu: origin (none) -> xyz=0.05 -0.01 0.15
- joint base_to_mainbar: origin (none) -> xyz=0.2 0.0 0.8
- joint base_to_platform: origin (none) -> xyz=-0.5 0.0 0.15
- joint base_to_sonar: origin (none) -> xyz=0.3 0.0 0.3
- joint frame_to_laser: origin (none) -> xyz=0.1 0.0 0.0
- joint mainbar_to_handbar: origin (none) -> xyz=0.0 0.0 0.7

Commit message: [URDF] rotate laser

File: code/ros-drivers/scoomatic_description/urdf/scoomatic.urdf (robot description, URDF)
Before this commit: robot scoomatic, 7 links, 6 joints
Joints:
- joint frame_to_laser: origin xyz=0.1 0.0 0.0 -> xyz=0.1 0.0 0.0 rpy=0.0 0.0 3.141592
